Commit message: modified mycobot_ros pkg for myCobot Pi

File: mycobot_description/urdf/mycobot/mycobot_urdf.urdf (robot description, URDF)
Before this commit: robot firefighter, 7 links, 6 joints
Links:
- link joint1: geometry visual mesh filename=package://myCobotROS/urdf/joint1.dae
- link joint2: geometry visual mesh filename=package://myCobotROS/urdf/joint2.dae
- link joint3: geometry visual mesh filename=package://myCobotROS/urdf/joint3.dae
- link joint4: geometry visual mesh filename=package://myCobotROS/urdf/joint4.dae
- link joint5: geometry visual mesh filename=package://myCobotROS/urdf/joint5.dae
- link joint6: geometry visual mesh filename=package://myCobotROS/urdf/joint6.dae
- link joint6_flange: geometry visual mesh filename=package://myCobotROS/urdf/joint7.dae
Joints:
- removed joint joint2_to_joint1
- removed joint joint3_to_joint2
- removed joint joint4_to_joint3
- removed joint joint5_to_joint4
- removed joint joint6_to_joint5
- removed joint joint6output_to_joint6
- added joint arm1_joint: type revolute, parent joint1, child joint2, origin xyz=0 0 0.13156 rpy=0 0 0, axis 0 0 1, limit lower=-3.14 upper=3.14159 effort=1000.0 velocity=0
- added joint arm2_joint: type revolute, parent joint2, child joint3, origin xyz=0 0  0 rpy=0 1.5708 -1.5708, axis 0 0 1, limit lower=-3.14 upper=3.14159 effort=1000.0 velocity=0
- added joint arm3_joint: type revolute, parent joint3, child joint4, origin xyz=  -0.1104 0 0    rpy=0 0 0, axis  0 0 1, limit lower=-3.14 upper=3.14159 effort=1000.0 velocity=0
- added joint arm4_joint: type revolute, parent joint4, child joint5, origin xyz=-0.096 0 0.06462 rpy=0 0 -1.5708, axis  0 0 1, limit lower=-3.14 upper=3.14159 effort=1000.0 velocity=0
- added joint arm5_joint: type revolute, parent joint5, child joint6, origin xyz=0 -0.07318 0 rpy=1.5708 -1.5708 0, axis 0 0 1, limit lower=-3.14 upper=3.14159 effort=1000.0 velocity=0
- added joint arm6_joint: type revolute, parent joint6, child joint6_flange, origin xyz=0 0.0456 0 rpy=-1.5708 0 0, axis 0 0 1, limit lower=-3.14 upper=3.14159 effort=1000.0 velocity=0

Commit message: fixed mycobot_description

File: mycobot_description/urdf/mycobot/mycobot_urdf.urdf (robot description, URDF)
Before this commit: robot firefighter, 7 links, 6 joints
Links:
- link joint1: geometry visual mesh filename=package://mycobot_description/urdf/mycobot/joint1.dae
- link joint2: geometry visual mesh filename=package://mycobot_description/urdf/mycobot/joint2.dae
- link joint3: geometry visual mesh filename=package://mycobot_description/urdf/mycobot/joint3.dae
- link joint4: geometry visual mesh filename=package://mycobot_description/urdf/mycobot/joint4.dae
- link joint5: geometry visual mesh filename=package://mycobot_description/urdf/mycobot/joint5.dae
- link joint6: geometry visual mesh filename=package://mycobot_description/urdf/mycobot/joint6.dae
- link joint6_flange: geometry visual mesh filename=package://mycobot_description/urdf/mycobot/joint7.dae
